File: hardware/LEDRibbonController.sch (KiCad schematic (older format))
At the start: 20 parts, among them J1 LED, J2 USB_OTG, J3 Battery, J4 ICSP, Q1 NTR4003NT1G, SW1 Mode, SW2 Power, U1 ATTINY10-TS, U2 MCP73831T-2ACI/OT

Commit message: Upgrade to kicad 5
Parts:
- removed J2: USB_OTG, Connectors:USB_Micro-B, symbol USB_OTG
- removed U1: ATTINY10-TS, TO_SOT_Packages_SMD:SOT-23-6, symbol ATTINY10-TS
- added J2: USB_B_Micro, Connector_USB:USB_Micro-B_Amphenol_10103594-0001LF_Horizontal, symbol Connector:USB_B_Micro
- added U1: ATtiny10-TS, Package_TO_SOT_SMD:SOT-23-6, symbol MCU_Microchip_ATtiny:ATtiny10-TS
- C1, C2, C3, C4: footprint Capacitors_SMD:C_0805_HandSoldering -> Capacitor_SMD:C_0805_2012Metric; symbol C -> LEDRibbonController-rescue:C
- D1, D2: footprint LEDs:LED_0805 -> LED_SMD:LED_0805_2012Metric_Pad1.15x1.40mm_HandSolder; symbol LED -> LEDRibbonController-rescue:LED
- J1: footprint Pin_Headers:Pin_Header_Straight_1x02_Pitch2.54mm -> Connector_PinHeader_2.54mm:PinHeader_1x02_P2.54mm_Vertical; symbol CONN_01X02 -> LEDRibbonController-rescue:CONN_01X02
- J3: symbol Battery_Cell -> LEDRibbonController-rescue:Battery_Cell
- J4: footprint Pin_Headers:Pin_Header_Straight_2x03_Pitch2.54mm -> Connector_PinHeader_2.54mm:PinHeader_2x03_P2.54mm_Vertical; symbol CONN_02X03 -> LEDRibbonController-rescue:CONN_02X03
- Q1: footprint TO_SOT_Packages_SMD:SOT-23 -> Package_TO_SOT_SMD:SOT-23; symbol MMBF170 -> LEDRibbonController-rescue:MMBF170
- R1, R2, R4, R5: footprint Resistors_SMD:R_0805_HandSoldering -> Resistor_SMD:R_0805_2012Metric_Pad1.15x1.40mm_HandSolder; symbol R -> LEDRibbonController-rescue:R
- R3: footprint Resistors_SMD:R_0805_HandSoldering -> Resistor_SMD:R_0805_2012Metric_Pad1.15x1.40mm_HandSolder; symbol R_Small -> LEDRibbonController-rescue:R_Small
- SW1: symbol SW_Push -> LEDRibbonController-rescue:SW_Push
- SW2: symbol SW_SPST -> LEDRibbonController-rescue:SW_SPST
- U2: symbol MCP73831T-2ACI/OT -> LEDRibbonController-rescue:MCP73831T-2ACI_OT
Connections:
- wire segments 61 -> 74
Other:
- moved on the sheet: C1, C2, J1, Q1, R1, R2, SW1

Commit message: Populate PCB with ALL THE NEW THINGS
Parts:
- removed J1: LED, Connector_PinHeader_2.54mm:PinHeader_1x02_P2.54mm_Vertical, symbol LEDRibbonController-rescue:CONN_01X02
- removed J4: ICSP, Connector_PinHeader_2.54mm:PinHeader_2x03_P2.54mm_Vertical, symbol LEDRibbonController-rescue:CONN_02X03
- removed U1: ATtiny10-TS, Package_TO_SOT_SMD:SOT-23-6, symbol MCU_Microchip_ATtiny:ATtiny10-TS
- added C4, C6: 4.7uF, Capacitor_SMD:C_0603_1608Metric_Pad1.05x0.95mm_HandSolder, symbol LEDRibbonController-rescue:C
- added C7: 10uF, Capacitor_SMD:C_0603_1608Metric_Pad1.05x0.95mm_HandSolder, symbol Device:C_Small
- added C8: 22uF, Capacitor_SMD:C_0603_1608Metric_Pad1.05x0.95mm_HandSolder, symbol Device:C_Small
- added D3, D4: 3v6, Diode_SMD:D_SOD-323, symbol Device:D_Zener_Small_ALT
- added D5, D6: 20V2A, Diode_SMD:D_SOD-323, symbol Device:D_Small
- added J1: PWM, Connector_PinHeader_2.54mm:PinHeader_1x04_P2.54mm_Vertical, symbol Connector_Generic:Conn_01x04
- added J4: ISP, Connector_PinHeader_2.54mm:PinHeader_2x03_P2.54mm_Vertical, symbol Connector:AVR-ISP-6
- added J5: Power, Connector_PinHeader_2.54mm:PinHeader_1x02_P2.54mm_Vertical, symbol Connector_Generic:Conn_01x02
- added L1: 2.2uH3A, Inductor_SMD:L_Vishay_IHLP-1212, symbol Device:L_Small
- added Q2, Q3: NTR4003NT1G, Package_TO_SOT_SMD:SOT-23, symbol LEDRibbonController-rescue:MMBF170
- added R10, R9: 68, Resistor_SMD:R_0603_1608Metric_Pad1.05x0.95mm_HandSolder, symbol Device:R
- added R12: 750K, Resistor_SMD:R_0603_1608Metric_Pad1.05x0.95mm_HandSolder, symbol Device:R_Small
- added R13: 100K, Resistor_SMD:R_0603_1608Metric_Pad1.05x0.95mm_HandSolder, symbol Device:R_Small
- added R4, R6: 20k, Resistor_SMD:R_0603_1608Metric_Pad1.05x0.95mm_HandSolder, symbol LEDRibbonController-rescue:R
- added R7: 2.2k, Resistor_SMD:R_0603_1608Metric_Pad1.05x0.95mm_HandSolder, symbol Device:R
- added U1: ATtiny85-20SU, Package_SO:SOIC-8_3.9x4.9mm_P1.27mm, symbol MCU_Microchip_ATtiny:ATtiny85-20SU
- added U3: PAM2401-8MSOP, Package_SO:MSOP-8_3x3mm_P0.65mm, symbol PAM2401:PAM2401-8MSOP
- C1: renamed from C2; footprint Capacitor_SMD:C_0805_2012Metric -> Capacitor_SMD:C_0603_1608Metric_Pad1.05x0.95mm_HandSolder
- C2: renamed from C1; footprint Capacitor_SMD:C_0805_2012Metric -> Capacitor_SMD:C_0603_1608Metric_Pad1.05x0.95mm_HandSolder
- C3: footprint Capacitor_SMD:C_0805_2012Metric -> Capacitor_SMD:C_0603_1608Metric_Pad1.05x0.95mm_HandSolder
- C5: renamed from C4; footprint Capacitor_SMD:C_0805_2012Metric -> Capacitor_SMD:C_0603_1608Metric_Pad1.05x0.95mm_HandSolder
- D1, D2: footprint LED_SMD:LED_0805_2012Metric_Pad1.15x1.40mm_HandSolder -> LED_SMD:LED_0603_1608Metric_Castellated
- R1, R2, R3: footprint Resistor_SMD:R_0805_2012Metric_Pad1.15x1.40mm_HandSolder -> Resistor_SMD:R_0603_1608Metric_Pad1.05x0.95mm_HandSolder
- R5: renamed from R4; footprint Resistor_SMD:R_0805_2012Metric_Pad1.15x1.40mm_HandSolder -> Resistor_SMD:R_0603_1608Metric
- R8: renamed from R5; value 470 -> 120; footprint Resistor_SMD:R_0805_2012Metric_Pad1.15x1.40mm_HandSolder -> Resistor_SMD:R_0603_1608Metric_Pad1.05x0.95mm_HandSolder
Connections:
- net labels added: +5V, +BATT, D+, D-, MISO, MOSI, PWM1, PWM2, PWM3, RST, SCK, Vin
- net labels removed: BATTERY, LED, RESET, TPICLK, TPIDATA
- wire segments 74 -> 152
- no-connect marks 4 -> 2
Other:
- moved on the sheet: C1, C2, C3, C5, D1, Q1, R1, R2, R3, R5, SW1, SW2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

Commit message: Remove VCC
Connections:
- net labels removed: VCC
Changed lines of the file:
@@
-$EndComp
-$Comp
-L LEDRibbonController-rescue:VCC #PWR05
-U 1 1 59C9D227
-P 650 4200
-F 0 "#PWR05" H 650 4050 50  0001 C CNN
-F 1 "VCC" H 650 4350 50  0000 C CNN
-F 2 "" H 650 4200 50  0001 C CNN
-F 3 "" H 650 4200 50  0001 C CNN
-	1    650  4200
-	1    0    0    -1
 $EndComp
 $Comp
@@
 	0    1    1    0
 $EndComp
-$Comp
-L LEDRibbonController-rescue:VCC #PWR016
-U 1 1 5B92C0FB
-P 2050 4200
-F 0 "#PWR016" H 2050 4050 50  0001 C CNN
-F 1 "VCC" H 2050 4350 50  0000 C CNN
-F 2 "" H 2050 4200 50  0001 C CNN
-F 3 "" H 2050 4200 50  0001 C CNN
-	1    2050 4200
-	1    0    0    -1
-$EndComp
 Wire Wire Line
 	2350 3850 2450 3850
@@
 	1    3700 4350
 	0    1    1    0
-$EndComp
-$Comp
-L LEDRibbonController-rescue:VCC #PWR018
-U 1 1 5B938E43
-P 3500 4200
-F 0 "#PWR018" H 3500 4050 50  0001 C CNN
-F 1 "VCC" H 3500 4350 50  0000 C CNN
-F 2 "" H 3500 4200 50  0001 C CNN
-F 3 "" H 3500 4200 50  0001 C CNN
-	1    3500 4200
-	1    0    0    -1
 $EndComp
 Wire Wire Line
@@
 Wire Wire Line
 	7800 3450 7800 3650
+$Comp
+L power:+5V #PWR?
+U 1 1 5BC46536
+P 650 4200
+F 0 "#PWR?" H 650 4050 50  0001 C CNN
+F 1 "+5V" H 665 4373 50  0000 C CNN
+F 2 "" H 650 4200 50  0001 C CNN
+F 3 "" H 650 4200 50  0001 C CNN
+	1    650  4200
+	1    0    0    -1
+$EndComp
+$Comp
+L power:+5V #PWR?
+U 1 1 5BC46D00
+P 2050 4200
+F 0 "#PWR?" H 2050 4050 50  0001 C CNN
+F 1 "+5V" H 2065 4373 50  0000 C CNN
+F 2 "" H 2050 4200 50  0001 C CNN
+F 3 "" H 2050 4200 50  0001 C CNN
+	1    2050 4200
+	1    0    0    -1
+$EndComp
+$Comp
+L power:+5V #PWR?
+U 1 1 5BC475A3
+P 3500 4200
+F 0 "#PWR?" H 3500 4050 50  0001 C CNN
+F 1 "+5V" H 3515 4373 50  0000 C CNN
+F 2 "" H 3500 4200 50  0001 C CNN
+F 3 "" H 3500 4200 50  0001 C CNN
+	1    3500 4200
+	1    0    0    -1
+$EndComp
 $EndSCHEMATC
