File: hardware/Attiny85/Big_18650/LitFist18650.sch (KiCad schematic (older format))
At the start: 41 parts, among them J1 PWM, J2 USB_B_Micro, J3 Battery, J4 ISP, Q1 NTR4003NT1G, Q2 NTR4003NT1G, Q3 NTR4003NT1G, SW1 Mode, SW2 Power, U1 ATtiny85-20SU, U2 MCP73831T-2ACI/OT, U3 PAM2401-8MSOP

Commit message: minor save
Parts:
- C1, C2, C3, C4, C5, C6: symbol LEDRibbonController-rescue:C -> LitFist18650-rescue:C-LEDRibbonController-rescue
- D1, D2: symbol LEDRibbonController-rescue:LED -> LitFist18650-rescue:LED-LEDRibbonController-rescue
- J3: symbol LEDRibbonController-rescue:Battery_Cell -> LitFist18650-rescue:Battery_Cell-LEDRibbonController-rescue
- Q1, Q2, Q3: symbol LEDRibbonController-rescue:MMBF170 -> LitFist18650-rescue:MMBF170-LEDRibbonController-rescue
- R1, R2, R4, R5, R6, R8: symbol LEDRibbonController-rescue:R -> LitFist18650-rescue:R-LEDRibbonController-rescue
- R3: symbol LEDRibbonController-rescue:R_Small -> LitFist18650-rescue:R_Small-LEDRibbonController-rescue
- SW1: symbol LEDRibbonController-rescue:SW_Push -> LitFist18650-rescue:SW_Push-LEDRibbonController-rescue
- SW2: symbol LEDRibbonController-rescue:SW_SPST -> LitFist18650-rescue:SW_SPST-LEDRibbonController-rescue
- U1: symbol MCU_Microchip_ATtiny:ATtiny85-20SU -> LitFist18650-rescue:ATtiny85-20SU-MCU_Microchip_ATtiny
- U2: symbol LEDRibbonController-rescue:MCP73831T-2ACI_OT -> LitFist18650-rescue:MCP73831T-2ACI_OT-LEDRibbonController-rescue
Changed lines of the file:
@@
 $EndDescr
 $Comp
-L LEDRibbonController-rescue:C C1
+L LitFist18650-rescue:C-LEDRibbonController-rescue C1
 U 1 1 59C9C8A6
 P 800 1600
@@
 $EndComp
 $Comp
-L LEDRibbonController-rescue:GND #PWR07
+L LitFist18650-rescue:GND-LEDRibbonController-rescue #PWR07
 U 1 1 59C9C999
 P 1650 2350
@@
 $EndComp
 $Comp
-L LEDRibbonController-rescue:MMBF170 Q1
+L LitFist18650-rescue:MMBF170-LEDRibbonController-rescue Q1
 U 1 1 59C9CEA8
 P 1350 3800
@@
 $EndComp
 $Comp
-L LEDRibbonController-rescue:R R2
+L LitFist18650-rescue:R-LEDRibbonController-rescue R2
 U 1 1 59C9CF55
 P 1050 4100
@@
 $EndComp
 $Comp
-L LEDRibbonController-rescue:GND #PWR03
+L LitFist18650-rescue:GND-LEDRibbonController-rescue #PWR03
 U 1 1 59C9CFCF
 P 1050 4400
@@
 $EndComp
 $Comp
-L LEDRibbonController-rescue:C C2
+L LitFist18650-rescue:C-LEDRibbonController-rescue C2
 U 1 1 59C9D1BD
 P 850 4350
@@
 $EndComp
 $Comp
-L LEDRibbonController-rescue:Battery_Cell J3
+L LitFist18650-rescue:Battery_Cell-LEDRibbonController-rescue J3
 U 1 1 59C9D408
 P 5800 1500
@@
 $EndComp
 $Comp
-L LEDRibbonController-rescue:GND #PWR09
+L LitFist18650-rescue:GND-LEDRibbonController-rescue #PWR09
 U 1 1 59C9D5B4
 P 5600 1750
@@
 $EndComp
 $Comp
-L LEDRibbonController-rescue:MCP73831T-2ACI_OT U2
+L LitFist18650-rescue:MCP73831T-2ACI_OT-LEDRibbonController-rescue U2
 U 1 1 59C9DDF2
 P 2400 6150
@@
 $EndComp
 $Comp
-L LEDRibbonController-rescue:GND #PWR02
+L LitFist18650-rescue:GND-LEDRibbonController-rescue #PWR02
 U 1 1 59C9E9ED
 P 3450 2150
@@
 $EndComp
 $Comp
-L LEDRibbonController-rescue:R R1
+L LitFist18650-rescue:R-LEDRibbonController-rescue R1
 U 1 1 59C9EA25
 P 3650 1850
@@
 $EndComp
 $Comp
-L LEDRibbonController-rescue:C C3
+L LitFist18650-rescue:C-LEDRibbonController-rescue C3
 U 1 1 59C9EFD0
 P 1100 6250
@@
 $EndComp
 $Comp
-L LEDRibbonController-rescue:LED D1
+L LitFist18650-rescue:LED-LEDRibbonController-rescue D1
 U 1 1 59C9F30F
 P 2300 5700
@@
 $EndComp
 $Comp
-L LEDRibbonController-rescue:R R5
+L LitFist18650-rescue:R-LEDRibbonController-rescue R5
 U 1 1 59C9F7BB
 P 2700 5700
@@
 $EndComp
 $Comp
-L LEDRibbonController-rescue:R_Small R3
+L LitFist18650-rescue:R_Small-LEDRibbonController-rescue R3
 U 1 1 59C9F949
 P 1550 6350
@@
 $EndComp
 $Comp
-L LEDRibbonController-rescue:GND #PWR010
+L LitFist18650-rescue:GND-LEDRibbonController-rescue #PWR010
 U 1 1 59C9FB34
 P 1100 6750
@@
 $EndComp
 $Comp
-L LEDRibbonController-rescue:GND #PWR08
+L LitFist18650-rescue:GND-LEDRibbonController-rescue #PWR08
 U 1 1 59C9FC10
 P 5850 4650
@@
 $EndComp
 $Comp
-L LEDRibbonController-rescue:C C5
+L LitFist18650-rescue:C-LEDRibbonController-rescue C5
 U 1 1 59C9FF60
 P 3300 6400
@@
 $EndComp
 $Comp
-L LEDRibbonController-rescue:GND #PWR015
+L LitFist18650-rescue:GND-LEDRibbonController-rescue #PWR015
 U 1 1 59CA0181
 P 3300 6750
@@
 $EndComp
 $Comp
-L LEDRibbonController-rescue:SW_SPST SW2
+L LitFist18650-rescue:SW_SPST-LEDRibbonController-rescue SW2
 U 1 1 59C9E171
 P 8250 3650
@@
 $EndComp
 $Comp
-L LEDRibbonController-rescue:GND #PWR011
+L LitFist18650-rescue:GND-LEDRibbonController-rescue #PWR011
 U 1 1 5B6A6B40
 P 1550 6750
@@
 	5750 4550 5850 4550
 $Comp
-L LEDRibbonController-rescue:LED D2
+L LitFist18650-rescue:LED-LEDRibbonController-rescue D2
 U 1 1 5B6A99E9
 P 7350 2550
@@
 $EndComp
 $Comp
-L LEDRibbonController-rescue:GND #PWR014
+L LitFist18650-rescue:GND-LEDRibbonController-rescue #PWR014
 U 1 1 5B6A9E89
 P 7650 2650
@@
 	7650 2550 7650 2650
 $Comp
-L LEDRibbonController-rescue:R R8
+L LitFist18650-rescue:R-LEDRibbonController-rescue R8
 U 1 1 5B6AAD79
 P 7000 2550
@@
 	9100 1000 9100 1100
 $Comp
-L LEDRibbonController-rescue:GND #PWR024
+L LitFist18650-rescue:GND-LEDRibbonController-rescue #PWR024
 U 1 1 5B8E5889
 P 9100 2100
@@
 	1450 4000 1450 4350
 $Comp
-L LEDRibbonController-rescue:MMBF170 Q2
+L LitFist18650-rescue:MMBF170-LEDRibbonController-rescue Q2
 U 1 1 5B92C0E3
 P 2750 3800
@@
 $EndComp
 $Comp
-L LEDRibbonController-rescue:R R4
+L LitFist18650-rescue:R-LEDRibbonController-rescue R4
 U 1 1 5B92C0E9
 P 2450 4100
@@
 $EndComp
 $Comp
-L LEDRibbonController-rescue:GND #PWR017
+L LitFist18650-rescue:GND-LEDRibbonController-rescue #PWR017
 U 1 1 5B92C0EF
 P 2450 4400
@@
 $EndComp
 $Comp
-L LEDRibbonController-rescue:C C4
+L LitFist18650-rescue:C-LEDRibbonController-rescue C4
 U 1 1 5B92C0F5
 P 2250 4350
@@
 PWM2
 $Comp
-L LEDRibbonController-rescue:MMBF170 Q3
+L LitFist18650-rescue:MMBF170-LEDRibbonController-rescue Q3
 U 1 1 5B938E2B
 P 4200 3800
@@
 $EndComp
 $Comp
-L LEDRibbonController-rescue:R R6
+L LitFist18650-rescue:R-LEDRibbonController-rescue R6
 U 1 1 5B938E31
 P 3900 4100
@@
 $EndComp
 $Comp
-L LEDRibbonController-rescue:GND #PWR019
+L LitFist18650-rescue:GND-LEDRibbonController-rescue #PWR019
 U 1 1 5B938E37
 P 3900 4400
@@
 $EndComp
 $Comp
-L LEDRibbonController-rescue:C C6
+L LitFist18650-rescue:C-LEDRibbonController-rescue C6
 U 1 1 5B938E3D
 P 3700 4350
@@
 Connection ~ 2750 1350
 $Comp
-L MCU_Microchip_ATtiny:ATtiny85-20SU U1
+L LitFist18650-rescue:ATtiny85-20SU-MCU_Microchip_ATtiny U1
 U 1 1 5B9F4534
 P 1650 1600
@@
 	8700 3650 8850 3650
 $Comp
-L LEDRibbonController-rescue:GND #PWR022
+L LitFist18650-rescue:GND-LEDRibbonController-rescue #PWR022
 U 1 1 5BA3B12B
 P 8700 3850
@@
 $EndComp
 $Comp
-L LEDRibbonController-rescue:GND #PWR026
+L LitFist18650-rescue:GND-LEDRibbonController-rescue #PWR026
 U 1 1 5BA44CCE
 P 10350 4050
@@
 Connection ~ 9900 4200
 $Comp
-L LEDRibbonController-rescue:GND #PWR025
+L LitFist18650-rescue:GND-LEDRibbonController-rescue #PWR025
 U 1 1 5BA66DE2
 P 9900 4400
@@
 	3250 1750 3250 1600
 $Comp
-L LEDRibbonController-rescue:SW_Push SW1
+L LitFist18650-rescue:SW_Push-LEDRibbonController-rescue SW1
 U 1 1 59C9E82C
 P 3800 1350
