File: STM32L0xx/hardware/18650/STM32L0xx_18650.kicad_pcb (KiCad board)
At the start: 2 copper layers, 50 parts, among them J1 Conn_ARM_JTAG_SWD_10, J2 Battery, J3 GPIO, J4 USB_B_Micro, J5 Power, J6 LEDs, J7 GPIO, Q1 BSS806N, Q2 BSS806N, Q3 BSS806N, Q4 BSS806N, SW1 Mode, SW2 Power, U1 STM32L052K8Tx, U2 AP2210N-3.3TRG1, U3 MCP73831T-2ACI/OT

Commit message: PCB for fab
Parts:
- removed C10, C12, C7, C8: 4.7uF, Capacitor_SMD:C_0603_1608Metric_Pad1.05x0.95mm_HandSolder
- removed J1: Conn_ARM_JTAG_SWD_10, Connector_PinHeader_1.27mm:PinHeader_2x05_P1.27mm_Vertical_SMD
- moved D1 52.3 mm to (75.7, 93.3)
- moved R1 21.8 mm to (127.7, 93.4)
- moved U2 20.3 mm to (105.0, 94.0), turned to 270 degrees
- moved D3 19.8 mm to (124.2, 93.4)
- moved D2 13.5 mm to (132.5, 93.2)
- moved C1 13.1 mm to (126.8, 106.5)
- moved R2 13.1 mm to (133.5, 106.5)
- moved R3 13.1 mm to (130.1, 106.5)
- moved C6 12.6 mm to (101.5, 93.0)
- moved D4 12.4 mm to (119.0, 93.0)
- moved R10 12.1 mm to (113.1, 97.9), turned to 0 degrees
- moved R8 12.0 mm to (116.7, 97.9), turned to 180 degrees
- moved R7 11.9 mm to (120.3, 97.9), turned to 180 degrees
- moved D7 11.8 mm to (112.2, 93.0), turned to 0 degrees
- moved R11 11.6 mm to (63.1, 93.4), turned to 180 degrees
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Connections:
- D4 pad 2: +BATT -> +3V3
- D5 pad 2: +BATT -> +3V3
- D7 pad 2: +BATT -> +3V3
- D8 pad 2: +BATT -> +3V3
- J3 pad 1: /PA8 -> /PA4
- J3 pad 2: /PA7 -> /PA5
- J3 pad 4: /PA5 -> /PA7
- J3 pad 5: /PA4 -> /PA8
Routing:
- net /VUSB: track 0.00 -> 88.4 mm, vias 0 -> 3
- net +3V3: track 0.00 -> 82.6 mm, vias 0 -> 7
- net Net-(D1-Pad1): track 0.00 -> 69.8 mm, vias 0 -> 1
- net +BATT: track 0.00 -> 53.5 mm, vias 0 -> 2
- net /BUTTON: track 0.00 -> 37.3 mm, vias 0 -> 2
- net /VIN: track 0.00 -> 37.2 mm, vias 0 -> 2
- net /USB_D-: track 0.00 -> 31.7 mm, vias 0 -> 2
- net /USB_D+: track 0.00 -> 31.7 mm, vias 0 -> 2
- net /PA4: track 0.00 -> 23.2 mm, vias 0 -> 1
- net /LED1: track 0.00 -> 23.0 mm, vias 0 -> 2
- net Net-(R2-Pad1): track 0.00 -> 22.6 mm
- net Net-(R11-Pad1): track 0.00 -> 20.8 mm, vias 0 -> 2
- net /LED2: track 0.00 -> 19.2 mm, vias 0 -> 2
- net /PA5: track 0.00 -> 18.9 mm, vias 0 -> 1
- net /PA9: track 0.00 -> 16.6 mm
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- added copper zone on B.Cu, net +3V3
- added copper zone on B.Cu, net +BATT
- added copper zone on F.Cu, net GND
Other:
- board outline added: 95.3 x 16 mm
- rule pad_to_mask_clearance: 0.051 -> 0.0508
- board text added: "PowerFist"
- board text added: "rev 2, 2019 Jeremy Gillick"

Commit message: Update hardware
Parts:
- added C10: 7pF, Capacitor_SMD:C_0603_1608Metric, F.Cu at (104.5, 99.6)
- added C7: 4.7uF, Capacitor_SMD:C_0603_1608Metric, F.Cu at (92.1, 103.0)
- added C8: 7pF, Capacitor_SMD:C_0603_1608Metric, F.Cu at (104.5, 103.7)
- added J1: SWD, Connector_PinHeader_1.27mm:PinHeader_1x03_P1.27mm_Vertical, F.Cu at (96.3, 106.2)
- added REF**: OSHW-Logo2_7.3x6mm_Copper, Symbol:OSHW-Logo2_7.3x6mm_Copper, B.Cu at (146.5, 104.5)
- added Y1: 32.768kHz, Crystal:Crystal_SMD_3215-2Pin_3.2x1.5mm, F.Cu at (104.9, 101.7)
- C1, C11, C2, C3, C4, C9: footprint Capacitor_SMD:C_0603_1608Metric_Pad1.05x0.95mm_HandSolder -> Capacitor_SMD:C_0603_1608Metric
- C5: value 100uf -> 100nf; footprint Capacitor_SMD:C_0603_1608Metric_Pad1.05x0.95mm_HandSolder -> Capacitor_SMD:C_0603_1608Metric
- C6: value 4.7uf -> 100nf; footprint Capacitor_SMD:C_0603_1608Metric_Pad1.05x0.95mm_HandSolder -> Capacitor_SMD:C_0603_1608Metric
- J2: moved to F.Cu
- J7: footprint Connector_PinHeader_2.54mm:PinHeader_1x04_P2.54mm_Vertical -> Connector_PinHeader_2.54mm:PinHeader_1x05_P2.54mm_Vertical
- R1: value 120 -> 330; footprint Resistor_SMD:R_0603_1608Metric_Pad1.05x0.95mm_HandSolder -> Resistor_SMD:R_0603_1608Metric
- R10, R12, R7, R8: value 300 -> 270; footprint Resistor_SMD:R_0603_1608Metric_Pad1.05x0.95mm_HandSolder -> Resistor_SMD:R_0603_1608Metric
- R11: value 470 -> 430
- R13, R2, R3, R4, R5, R6, R9: footprint Resistor_SMD:R_0603_1608Metric_Pad1.05x0.95mm_HandSolder -> Resistor_SMD:R_0603_1608Metric
- U1: value STM32L052K8Tx -> STM32L072CBTx; footprint Package_QFP:LQFP-32_7x7mm_P0.8mm -> Package_QFP:LQFP-48_7x7mm_P0.5mm
- U2: value AP2210N-3.3TRG1 -> AP2210-3.3TRG1
- moved D1 18.2 mm to (62.0, 105.2), turned to 0 degrees
- moved U2 17.8 mm to (88.2, 99.8), turned to 0 degrees
- moved C6 12.5 mm to (104.5, 105.2), turned to 0 degrees
- moved L1 10.5 mm to (106.0, 94.0), turned to 90 degrees
- moved C9 9.36 mm to (79.0, 99.7), turned to 270 degrees
- moved D3 9.25 mm to (133.5, 93.4), turned to 180 degrees
- moved C2 9.05 mm to (103.0, 94.0), turned to 90 degrees
- moved J7 7.60 mm to (79.7, 105.6), turned to 90 degrees
- moved C3 7.40 mm to (104.5, 93.9), turned to 90 degrees
- moved D2 6.40 mm to (126.1, 93.3)
- moved R1 2.25 mm to (130.0, 93.4), turned to 180 degrees
- moved C4 2.06 mm to (104.5, 106.8), turned to 0 degrees
- moved C11 2.05 mm to (85.6, 99.7)
- moved R6 2.05 mm to (81.6, 102.4)
- moved U3 2.05 mm to (82.3, 99.8)
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Connections:
- C2 pad 1: /VDDA -> Net-(C2-Pad1)
- C3 pad 1: /VDDA -> Net-(C2-Pad1)
- D1 pad 1: Net-(D1-Pad1) -> /VUSB
- D1 pad 2: /VUSB -> Net-(D1-Pad2)
- D2 pad 1: Net-(D1-Pad1) -> /VUSB
- J4 pad 1: /VUSB -> Net-(D1-Pad2)
- J7 pad 1: /PB7 -> /PA9
- J7 pad 2: /PB6 -> /PA10
- J7 pad 3: /PA10 -> /PB6
- J7 pad 4: /PA9 -> /PB7
- L1 pad 1: +3V3 -> Net-(C2-Pad1)
- L1 pad 2: /VDDA -> +3V3
- SW2 pad 1: Net-(D1-Pad1) -> /VUSB
- U1 pad 10: /PA4 -> /LED1
- U1 pad 11: /PA5 -> /LED2
- U1 pad 12: /PA6 -> /LED3
- U1 pad 13: /PA7 -> /LED4
- U1 pad 14: (no net) -> /PA4
- U1 pad 15: (no net) -> /PA5
- U1 pad 16: GND -> /PA6
- U1 pad 17: +3V3 -> /PA7
- U1 pad 18: /PA8 -> (no net)
- U1 pad 19: /PA9 -> (no net)
- U1 pad 20: /PA10 -> (no net)
- U1 pad 21: /USB_D- -> (no net)
- U1 pad 22: /USB_D+ -> (no net)
- U1 pad 23: /SWDIO -> GND
- U1 pad 24: /SWCLK -> +3V3
- U1 pad 27: /BUTTON -> (no net)
- U1 pad 29: /PB6 -> /PA8
- U1 pad 3: (no net) -> Net-(C8-Pad1)
- U1 pad 30: /PB7 -> /PA9
- U1 pad 31: /BUTTON -> /PA10
- U1 pad 32: GND -> /USB_D-
- U1 pad 4: /RESET -> Net-(C10-Pad1)
- U1 pad 5: /VDDA -> (no net)
- U1 pad 6: /LED1 -> (no net)
- U1 pad 7: /LED2 -> /RESET
- U1 pad 8: /LED3 -> GND
- U1 pad 9: /LED4 -> Net-(C2-Pad1)
Routing:
- net Net-(D1-Pad1): track 69.8 -> 0.00 mm, vias 1 -> 0
- net GND: track 3.37 -> 51.6 mm, vias 0 -> 14
- net /VUSB: track 88.4 -> 130.4 mm, vias 3 -> 2
- net +3V3: track 82.6 -> 52.6 mm, vias 7 -> 10
- net /VIN: track 37.2 -> 56.9 mm
- net +BATT: track 53.5 -> 70.7 mm, vias 2 -> 1
- net /PB8: track 0.00 -> 10.4 mm
- net Net-(D1-Pad2): track 0.00 -> 10.0 mm
- net /RESET: track 0.00 -> 9.44 mm
- net Net-(C2-Pad1): track 0.00 -> 8.35 mm
- net /SWDIO: track 0.00 -> 7.12 mm, vias 0 -> 1
- net /VDDA: track 6.84 -> 0.00 mm
- net /SWCLK: track 0.00 -> 5.91 mm, vias 0 -> 1
- net Net-(C10-Pad1): track 0.00 -> 5.55 mm
- net Net-(C8-Pad1): track 0.00 -> 4.23 mm
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- added copper zone on PWR, net +3V3
- added copper zone on PWR, net +BATT
- added copper zone on GND, net GND
- removed copper zone on B.Cu, net +3V3
- removed copper zone on B.Cu, net +BATT
- removed copper zone on F.Cu, net GND
Other:
- board size 95.3 x 16 mm -> 108.4 x 16 mm
- copper layers 2 -> 4
- net class Default: clearance 0.1524 -> 0.127; trace_width 0.1524 -> 0.127; via_dia 0.6858 -> 0.4572; via_drill 0.3302 -> 0.254
- rule trace_clearance: 0.1524 -> 0.127
- rule trace_min: 0.1524 -> 0.127
- rule via_min_size: 0.508 -> 0.4572
- board text added: "(max 2.3A per channel!)"
- board text added: "3.3v"
- board text added: "Batt+"
- board text added: "CLK"
- board text added: "Gnd"
- board text added: "IO"
- board text added: "PA0"
- board text added: "PA1"
- board text added: "PA10"
- board text added: "PA2"
- board text added: "PA3"
- board text added: "PA4"
- board text added: "PA5"
- board text added: "PA6"
- board text added: "PA7"
- board text added: "PA8"
- board text added: "PA9"
- board text added: "PB6"
- board text added: "PB7"
- board text added: "PB8"
- board text added: "PWM / LEDs"
- board text added: "Power"
- board text added: "RESET"
- board text added: "USB+"
- board text added: "pArm board"
- board text added: "v1 Jeremy Gillick"
- board text removed: "PowerFist"
- board text removed: "rev 2, 2019 Jeremy Gillick"
