File: STM32L0xx/hardware/18650/STM32L0xx_18650.sch (KiCad schematic (older format))
At the start: 49 parts

Commit message: Annotations
Parts:
- gave numbers to parts that had none: 49
Other:
- moved on the sheet: U2

Commit message: Update LED circuit
Parts:
- removed C10, C12, C7, C8: 4.7uF, Capacitor_SMD:C_0603_1608Metric_Pad1.05x0.95mm_HandSolder, symbol Device:C_Small
- added J7: GPIO, Connector_PinHeader_2.54mm:PinHeader_1x04_P2.54mm_Vertical, symbol Connector_Generic:Conn_01x04
- J2: footprint Jeremy:Battery_Clips_8650 -> Jeremy:Battery_Clips_18650
- J3: value Headers -> GPIO; footprint Connector_PinHeader_2.54mm:PinHeader_1x09_P2.54mm_Vertical -> Connector_PinHeader_2.54mm:PinHeader_1x05_P2.54mm_Vertical; symbol Connector_Generic:Conn_01x09 -> Connector_Generic:Conn_01x05
- J4: footprint (none) -> Jeremy:USB_Micro-B_Amphenol_10103594-0001LF_Horizontal
- J6: value PWM -> LEDs
- U3: footprint SOT95P280X145-5N -> Package_TO_SOT_SMD:SOT-23-5_HandSoldering; Digikey (none) -> MCP73831T-2ACI/OTCT-ND
Connections:
- net VDD is gone; now on net +3V3: U1.1 (VDD), U1.17 (VDD)
- net +3V3: now also D4.2 (A), D5.2 (A), D7.2 (A), D8.2 (A), J5.3 (Pin_3); no longer J5.4 (Pin_4)
- net +BATT: now also J5.4 (Pin_4); no longer D4.2 (A), D5.2 (A), D7.2 (A), D8.2 (A), J5.3 (Pin_3)
- net PA10: now also J7.3 (Pin_3); no longer J3.3 (Pin_3)
- net PA4: now also J3.5 (Pin_5); no longer J3.9 (Pin_9)
- net PA5: now also J3.4 (Pin_4); no longer J3.8 (Pin_8)
- net PA6: now also J3.3 (Pin_3); no longer J3.7 (Pin_7)
- net PA7: now also J3.2 (Pin_2); no longer J3.6 (Pin_6)
- net PA8: now also J3.1 (Pin_1); no longer J3.5 (Pin_5)
- net PA9: now also J7.4 (Pin_4); no longer J3.4 (Pin_4)
- net PB6: now also J7.2 (Pin_2); no longer J3.2 (Pin_2)
- net PB7: now also J7.1 (Pin_1); no longer J3.1 (Pin_1)
- net VDDA: now also C2.1, C3.1, L1.2
- net VIN: no longer C9.1, D6.2 (A), U3.4 (VDD)
- net VUSB: now also C9.1, D6.2 (A), U3.4 (VDD)
- net JTAG_TDI: no longer names the net of J1.8 (NC/TDI)
- net SWO: no longer names the net of J1.6 (SWO/TDO)
- no-connect marks 1 -> 10
Other:
- moved on the sheet: D4, D5, D7, D8, J6, Q1, Q2, Q3, Q4, R10, R12, R13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

Commit message: Update hardware
Parts:
- removed D2: 20V2A, Diode_SMD:D_SOD-323_HandSoldering, symbol Device:D_Small
- removed J1: Conn_ARM_JTAG_SWD_10, Connector_PinHeader_1.27mm:PinHeader_2x05_P1.27mm_Vertical_SMD, symbol Connector:Conn_ARM_JTAG_SWD_10
- removed U1: STM32L052K8Tx, Package_QFP:LQFP-32_7x7mm_P0.8mm, symbol MCU_ST_STM32L0:STM32L052K8Tx
- removed U2: AP2210N-3.3TRG1, Package_TO_SOT_SMD:SOT-23, symbol Regulator_Linear:AP2210N-3.3TRG1
- added C10, C8: 7pF, Capacitor_SMD:C_0603_1608Metric, symbol Device:C_Small
- added C7: 4.7uF, Capacitor_SMD:C_0603_1608Metric, symbol Device:C_Small
- added D2: 20V2A, Diode_SMD:D_SOD-323, symbol Device:D_Schottky_Small
- added J1: Debug, Connector_PinHeader_1.27mm:PinHeader_1x03_P1.27mm_Vertical, symbol Connector_Generic:Conn_01x03
- added U1: STM32L072CBTx, Package_QFP:LQFP-48_7x7mm_P0.5mm, symbol MCU_ST_STM32L0:STM32L072CBTx
- added U2: AP2210N-3.3TRG1, Package_TO_SOT_SMD:SOT-23, symbol Jeremy:AP2210-3.3TRG1
- added Y1: 32.768kHz, Crystal:Crystal_SMD_3215-2Pin_3.2x1.5mm, symbol Device:Crystal_Small
- C1: footprint Capacitor_SMD:C_0603_1608Metric_Pad1.05x0.95mm_HandSolder -> Capacitor_SMD:C_0603_1608Metric; MPN (none) -> MF-CAP-0603-0.1uF; Package (none) -> 0603
- C11: footprint Capacitor_SMD:C_0603_1608Metric_Pad1.05x0.95mm_HandSolder -> Capacitor_SMD:C_0603_1608Metric; symbol LitFist18650-rescue:C-LEDRibbonController-rescue -> Device:C; MPN (none) -> KEMET C0603C475K9PACTU; Package (none) -> 0603
- C2: footprint Capacitor_SMD:C_0603_1608Metric_Pad1.05x0.95mm_HandSolder -> Capacitor_SMD:C_0603_1608Metric; MPN (none) -> MF-CAP-0603-1uF; Package (none) -> 0603
- C3: footprint Capacitor_SMD:C_0603_1608Metric_Pad1.05x0.95mm_HandSolder -> Capacitor_SMD:C_0603_1608Metric; MFN (none) -> CC0603KRX7R9BB103; MPN (none) -> Yageo; Package (none) -> 0603
- C4: footprint Capacitor_SMD:C_0603_1608Metric_Pad1.05x0.95mm_HandSolder -> Capacitor_SMD:C_0603_1608Metric; MFN (none) -> AVX; MPN (none) -> 06035C104K4T2A; Package (none) -> 0603
- C5: value 100uf -> 100nf; footprint Capacitor_SMD:C_0603_1608Metric_Pad1.05x0.95mm_HandSolder -> Capacitor_SMD:C_0603_1608Metric; MFN (none) -> AVX; MPN (none) -> 06035C104K4T2A; Package (none) -> 0603
- C6: value 4.7uf -> 100nf; footprint Capacitor_SMD:C_0603_1608Metric_Pad1.05x0.95mm_HandSolder -> Capacitor_SMD:C_0603_1608Metric; MFN (none) -> AVX; MPN (none) -> 06035C104K4T2A; Package (none) -> 0603
- C9: symbol LitFist18650-rescue:C-LEDRibbonController-rescue -> Device:C; MPN (none) -> KEMET C0603C475K9PACTU; Package (none) -> 0603
- D1: footprint Diode_SMD:D_SOD-323_HandSoldering -> Diode_SMD:D_SOD-323; symbol Device:D_Small -> Device:D_Schottky_Small; MPN (none) -> SMD22WS-TP
- D3: symbol LitFist18650-rescue:LED-LEDRibbonController-rescue -> Device:LED; MFN (none) -> Rohm; MPN (none) -> SML-D12V1WT86; Package (none) -> 0603
- D4, D5, D7, D8: footprint LED_SMD:LED_0603_1608Metric_Pad1.05x0.95mm_HandSolder -> LED_SMD:LED_0603_1608Metric; MPN (none) -> 150060VS75000; Package (none) -> 0603
- D6: symbol LitFist18650-rescue:LED-LEDRibbonController-rescue -> Device:LED; MPN (none) -> 150060VS75000; Package (none) -> 0603
- J2: symbol LitFist18650-rescue:Battery_Cell-LEDRibbonController-rescue -> Device:Battery_Cell; Digikey (none) -> 36-54-ND; MFN (none) -> Keystone Electronics; MPN (none) -> Keystone 54
- J4: MFN (none) -> Amphenol; MPN (none) -> 10103594-0001LF
- J7: footprint Connector_PinHeader_2.54mm:PinHeader_1x04_P2.54mm_Vertical -> Connector_PinHeader_2.54mm:PinHeader_1x05_P2.54mm_Vertical; symbol Connector_Generic:Conn_01x04 -> Connector_Generic:Conn_01x05
- L1: footprint Inductor_SMD:L_0603_1608Metric_Pad1.05x0.95mm_HandSolder -> Inductor_SMD:L_0603_1608Metric; Digikey 1276-6355-1-ND -> 490-9702-1-ND; MFN CIC10J601NC -> (none); MPN (none) -> BLM18TG601TN1D
- Q1, Q2, Q3, Q4: symbol LitFist18650-rescue:MMBF170-LEDRibbonController-rescue -> Transistor_FET:MMBF170; MPN (none) -> BSS806NH6327XTSA1
- R1: value 120 -> 270; footprint Resistor_SMD:R_0603_1608Metric_Pad1.05x0.95mm_HandSolder -> Resistor_SMD:R_0603_1608Metric; symbol LitFist18650-rescue:R-LEDRibbonController-rescue -> Device:R; Package (none) -> 0603
- R10, R12, R7, R8: value 300 -> 270; footprint Resistor_SMD:R_0603_1608Metric_Pad1.05x0.95mm_HandSolder -> Resistor_SMD:R_0603_1608Metric; MPN (none) -> CRCW0603270RJNEA; Package (none) -> 0603
- R11: value 470 -> 430; symbol LitFist18650-rescue:R-LEDRibbonController-rescue -> Device:R; MPN (none) -> ERJ-PA3F4300V; Package (none) -> 0603
- R13, R2, R4, R5, R9: footprint Resistor_SMD:R_0603_1608Metric_Pad1.05x0.95mm_HandSolder -> Resistor_SMD:R_0603_1608Metric; symbol LitFist18650-rescue:R-LEDRibbonController-rescue -> Device:R; MPN (none) -> CR0603-FX-2002ELF; Package (none) -> 0603
- R3: footprint Resistor_SMD:R_0603_1608Metric_Pad1.05x0.95mm_HandSolder -> Resistor_SMD:R_0603_1608Metric; MPN (none) -> MF-RES-0603-330; Package (none) -> 0603
- R6: footprint Resistor_SMD:R_0603_1608Metric_Pad1.05x0.95mm_HandSolder -> Resistor_SMD:R_0603_1608Metric; symbol LitFist18650-rescue:R_Small-LEDRibbonController-rescue -> Device:R_Small; Package (none) -> 0603
- SW1: symbol LitFist18650-rescue:SW_Push-LEDRibbonController-rescue -> Switch:SW_Push; MFN (none) -> TE Connectivity; MPN FSMSM -> 1437566-3
- SW2: symbol LitFist18650-rescue:SW_SPST-LEDRibbonController-rescue -> Switch:SW_SPST
- U3: symbol LitFist18650-rescue:MCP73831T-2ACI_OT-LEDRibbonController-rescue -> STM32L0xx_18650-rescue:MCP73831T-2ACI_OT-LEDRibbonController-rescue-LitFist18650-rescue
Connections:
- net +3V3: now also L1.2, C7.1, U1.1 (VDD), U1.24 (VDD), U1.36 (VDD_USB), U1.48 (VDD), U2.2 (VOUT); no longer L1.1
- net +BATT: now also D2.2 (A)
- net BUTTON: now also U1.40 (PB4), U1.44 (BOOT0)
- net GND: now also C10.2, C7.2, C8.2, U1.23 (VSS), U1.35 (VSS), U1.47 (VSS), U1.8 (VSSA), U2.1 (GND)
- net LED1: now also U1.10 (PA0)
- net LED2: now also U1.11 (PA1)
- net LED3: now also U1.12 (PA2)
- net LED4: now also U1.13 (PA3)
- net PA10: now also J7.2 (Pin_2), U1.31 (PA10); no longer J7.3 (Pin_3)
- net PA4: now also J3.1 (Pin_1), U1.14 (PA4); no longer J3.5 (Pin_5)
- net PA5: now also J3.2 (Pin_2), U1.15 (PA5); no longer J3.4 (Pin_4)
- net PA6: now also U1.16 (PA6)
- net PA7: now also J3.4 (Pin_4), U1.17 (PA7); no longer J3.2 (Pin_2)
- net PA8: now also J3.5 (Pin_5), U1.29 (PA8); no longer J3.1 (Pin_1)
- net PA9: now also J7.1 (Pin_1), U1.30 (PA9); no longer J7.4 (Pin_4)
- net PB6: now also J7.3 (Pin_3), U1.42 (PB6); no longer J7.2 (Pin_2)
- net PB7: now also J7.4 (Pin_4), U1.43 (PB7); no longer J7.1 (Pin_1)
- net RESET: now also J1.3 (Pin_3), U1.7 (NRST)
- net SWCLK: now also J1.2 (Pin_2), U1.37 (PA14)
- net SWDIO: now also J1.1 (Pin_1), U1.34 (PA13)
- net USB_D+: now also U1.33 (PA12)
- net USB_D-: now also U1.32 (PA11)
- net VIN: now also U2.3 (VIN)
- net VUSB: now also D1.1 (K), SW2.1 (A), D2.1 (K); no longer D1.2 (A), J4.1 (VBUS)
- net VDDA: no longer names the net of C2.1, C3.1
- net VDDA: now also L1.1, U1.9 (VDDA); no longer L1.2
- new net: D1.2 (A), J4.1 (VBUS)
- new net: C8.1, U1.3 (PC14), Y1.1
- new net: C10.1, U1.4 (PC15), Y1.2
- new net PB8: J7.5 (Pin_5), U1.45 (PB8)
- no-connect marks 10 -> 17
Other:
- note added: "TODO: ^ Add diode here\n(PMEG045T100EPDAZ)"
- note removed: "JTAG Connector"
- note removed: "STM32 Decoupling Caps"
- moved on the sheet: C1, C11, C2, C3, C4, C5, C6, J2, J3, J5, L1, R1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
