File: hardware/STM32L0xx/STM32L0xx_18650.kicad_pcb (KiCad board)
At the start: 4 copper layers, 108.4 x 16 mm, 50 parts, among them J1 SW Debug, J2 Battery, J3 GPIO, J4 USB_B_Micro, J5 Power, J6 LEDs, J7 GPIO, Q1 BSS806N, Q2 BSS806N, Q3 BSS806N, Q4 BSS806N, SW1 Mode, SW2 Power, U1 STM32L072KZTx, U2 AP2210N-3.3TRG1, U3 MCP73833-AMI_UN, Y1 32.768kHz

Commit message: Make PCB labels bigger. Export gerbers.
Other:
- board text added: "rev 1a2"
- board text removed: "rev 1a"
Changed lines of the file:
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@@
     (38 B.Mask user)
     (39 F.Mask user)
-    (40 Dwgs.User user hide)
+    (40 Dwgs.User user)
     (41 Cmts.User user)
     (42 Eco1.User user)
@@
       (effects (font (size 0.7 0.7) (thickness 0.1)))
     )
-    (fp_text user "Battery with built-in protection required" (at 0 1.27) (layer B.SilkS)
-      (effects (font (size 0.5 0.5) (thickness 0.08)) (justify mirror))
+    (fp_text user "Built-in protection circuit required" (at 0 1.27) (layer B.SilkS)
+      (effects (font (size 0.6 0.55) (thickness 0.08)) (justify mirror))
     )
     (fp_line (start -22.22 -5.6) (end -22.22 5.6) (layer F.CrtYd) (width 0.15))
@@
       (effects (font (size 1 1) (thickness 0.15)))
     )
-    (fp_text value "SW Debug" (at 2.325 2.55 180) (layer B.SilkS)
-      (effects (font (size 0.5 0.5) (thickness 0.1)) (justify mirror))
+    (fp_text value "SW Debug" (at 2.45 2.575 180) (layer B.SilkS)
+      (effects (font (size 0.65 0.65) (thickness 0.1)) (justify mirror))
     )
     (fp_line (start -0.2175 -0.635) (end 2.34 -0.635) (layer F.Fab) (width 0.1))
@@
     (effects (font (size 1 1) (thickness 0.2)))
   )
-  (gr_text "rev 1a" (at 152.5 96.525) (layer B.SilkS)
+  (gr_text "rev 1a2" (at 152.5 96.525) (layer B.SilkS)
     (effects (font (size 0.75 0.75) (thickness 0.1)) (justify left mirror))
   )
-  (gr_text "GND  USB+  3.3v  Batt+" (at 116.775 107.45) (layer F.SilkS)
-    (effects (font (size 0.5 0.5) (thickness 0.1)))
-  )
-  (gr_text "PA8  PA7  PA6  PA5  PA4" (at 84.8 93.575 180) (layer F.SilkS)
-    (effects (font (size 0.6 0.6) (thickness 0.1)))
-  )
-  (gr_text "PA9  PA10  PB5  PB6  PB7" (at 84.85 107.45) (layer F.SilkS)
-    (effects (font (size 0.54 0.54) (thickness 0.1)))
+  (gr_text "GND USB+ 3.3v Batt+" (at 116.95 107.45) (layer F.SilkS)
+    (effects (font (size 0.62 0.62) (thickness 0.1)))
+  )
+  (gr_text "PA8 PA7 PA6 PA5 PA4" (at 84.8 93.5 180) (layer F.SilkS)
+    (effects (font (size 0.65 0.7) (thickness 0.1)))
+  )
+  (gr_text "PA9 PA10 PB5 PB6 PB7" (at 84.85 107.45) (layer F.SilkS)
+    (effects (font (size 0.65 0.65) (thickness 0.1)))
   )
   (gr_text JTAG (at 93.425 105.575 90) (layer F.SilkS)
-    (effects (font (size 0.5 0.5) (thickness 0.1)))
+    (effects (font (size 0.65 0.65) (thickness 0.1)))
   )
   (gr_text "Created by Jeremy Gillick" (at 145.825 105.375) (layer B.SilkS)
     (effects (font (size 0.75 0.75) (thickness 0.1)) (justify mirror))
   )
-  (gr_text "(max 2.3A per channel!)" (at 114 98.05) (layer B.SilkS)
-    (effects (font (size 0.4 0.4) (thickness 0.06)) (justify mirror))
+  (gr_text "(max 2.3A per channel!)" (at 115.25 98.3) (layer B.SilkS)
+    (effects (font (size 0.55 0.55) (thickness 0.06)) (justify mirror))
   )
   (gr_line (start 156.6 92) (end 158.499999 91.999845) (layer Edge.Cuts) (width 0.15))
@@
   (gr_arc (start 60.1 106) (end 58.1 106) (angle -90) (layer Edge.Cuts) (width 0.15))
   (gr_arc (start 60.1 94) (end 60.1 92) (angle -90) (layer Edge.Cuts) (width 0.15))
-  (gr_text PA8 (at 89.875 97.2) (layer B.SilkS)
-    (effects (font (size 0.5 0.5) (thickness 0.1)) (justify mirror))
-  )
-  (gr_text PA7 (at 87.375 97.2) (layer B.SilkS)
-    (effects (font (size 0.5 0.5) (thickness 0.1)) (justify mirror))
-  )
-  (gr_text PA6 (at 84.8 97.2) (layer B.SilkS)
-    (effects (font (size 0.5 0.5) (thickness 0.1)) (justify mirror))
-  )
-  (gr_text PA5 (at 82.225 97.175) (layer B.SilkS)
-    (effects (font (size 0.5 0.5) (thickness 0.1)) (justify mirror))
-  )
-  (gr_text PA4 (at 79.675 97.2) (layer B.SilkS)
-    (effects (font (size 0.5 0.5) (thickness 0.1)) (justify mirror))
-  )
-  (gr_text PB8 (at 89.85 103.925) (layer B.SilkS)
-    (effects (font (size 0.5 0.5) (thickness 0.1)) (justify mirror))
-  )
-  (gr_text PB7 (at 87.325 103.925) (layer B.SilkS)
-    (effects (font (size 0.5 0.5) (thickness 0.1)) (justify mirror))
-  )
-  (gr_text PB6 (at 84.75 103.95) (layer B.SilkS)
-    (effects (font (size 0.5 0.5) (thickness 0.1)) (justify mirror))
-  )
-  (gr_text PA10 (at 82.25 103.95) (layer B.SilkS)
-    (effects (font (size 0.5 0.5) (thickness 0.1)) (justify mirror))
-  )
-  (gr_text PA9 (at 79.725 103.975) (layer B.SilkS)
-    (effects (font (size 0.5 0.5) (thickness 0.1)) (justify mirror))
+  (gr_text PA8 (at 89.85 97.4) (layer B.SilkS)
+    (effects (font (size 0.65 0.65) (thickness 0.1)) (justify mirror))
+  )
+  (gr_text PA7 (at 87.375 97.4) (layer B.SilkS)
+    (effects (font (size 0.65 0.65) (thickness 0.1)) (justify mirror))
+  )
+  (gr_text PA6 (at 84.8 97.4) (layer B.SilkS)
+    (effects (font (size 0.65 0.65) (thickness 0.1)) (justify mirror))
+  )
+  (gr_text PA5 (at 82.2 97.4) (layer B.SilkS)
+    (effects (font (size 0.65 0.65) (thickness 0.1)) (justify mirror))
+  )
+  (gr_text PA4 (at 79.65 97.4) (layer B.SilkS)
+    (effects (font (size 0.65 0.65) (thickness 0.1)) (justify mirror))
+  )
+  (gr_text PB8 (at 89.85 103.85) (layer B.SilkS)
+    (effects (font (size 0.65 0.65) (thickness 0.1)) (justify mirror))
+  )
+  (gr_text PB7 (at 87.325 103.85) (layer B.SilkS)
+    (effects (font (size 0.65 0.65) (thickness 0.1)) (justify mirror))
+  )
+  (gr_text PB6 (at 84.75 103.85) (layer B.SilkS)
+    (effects (font (size 0.65 0.65) (thickness 0.1)) (justify mirror))
+  )
+  (gr_text PA10 (at 82.25 103.85) (layer B.SilkS)
+    (effects (font (size 0.65 0.65) (thickness 0.1)) (justify mirror))
+  )
+  (gr_text PA9 (at 79.725 103.85) (layer B.SilkS)
+    (effects (font (size 0.65 0.65) (thickness 0.1)) (justify mirror))
   )
   (gr_text PA3 (at 110.1 97.175) (layer B.SilkS)
-    (effects (font (size 0.5 0.5) (thickness 0.1)) (justify mirror))
+    (effects (font (size 0.65 0.65) (thickness 0.1)) (justify mirror))
   )
   (gr_text PA2 (at 112.65 97.175) (layer B.SilkS)
-    (effects (font (size 0.5 0.5) (thickness 0.1)) (justify mirror))
+    (effects (font (size 0.65 0.65) (thickness 0.1)) (justify mirror))
   )
   (gr_text PA1 (at 115.2 97.175) (layer B.SilkS)
-    (effects (font (size 0.5 0.5) (thickness 0.1)) (justify mirror))
+    (effects (font (size 0.65 0.65) (thickness 0.1)) (justify mirror))
   )
   (gr_text PA0 (at 117.75 97.2) (layer B.SilkS)
-    (effects (font (size 0.5 0.5) (thickness 0.1)) (justify mirror))
-  )
-  (gr_text Batt+ (at 120.25 97.125) (layer B.SilkS)
-    (effects (font (size 0.5 0.5) (thickness 0.1)) (justify mirror))
+    (effects (font (size 0.65 0.65) (thickness 0.1)) (justify mirror))
+  )
+  (gr_text Batt+ (at 120.5 97.125) (layer B.SilkS)
+    (effects (font (size 0.65 0.65) (thickness 0.1)) (justify mirror))
   )
   (gr_text "PWM / LEDs" (at 115.25 93.525) (layer B.SilkS)
     (effects (font (size 1 1) (thickness 0.2)) (justify mirror))
   )
-  (gr_text Batt+ (at 120.275 103.9) (layer B.SilkS)
-    (effects (font (size 0.5 0.5) (thickness 0.1)) (justify mirror))
+  (gr_text Batt+ (at 120.55 103.9) (layer B.SilkS)
+    (effects (font (size 0.65 0.6) (thickness 0.1)) (justify mirror))
   )
   (gr_text 3.3v (at 117.775 103.925) (layer B.SilkS)
-    (effects (font (size 0.5 0.5) (thickness 0.1)) (justify mirror))
-  )
-  (gr_text USB+ (at 115.25 103.925) (layer B.SilkS)
-    (effects (font (size 0.5 0.5) (thickness 0.1)) (justify mirror))
+    (effects (font (size 0.65 0.6) (thickness 0.1)) (justify mirror))
+  )
+  (gr_text USB+ (at 115.05 103.925) (layer B.SilkS)
+    (effects (font (size 0.65 0.6) (thickness 0.1)) (justify mirror))
   )
   (gr_text Gnd (at 112.7 103.925) (layer B.SilkS)
-    (effects (font (size 0.5 0.5) (thickness 0.1)) (justify mirror))
-  )
-  (gr_text Power (at 116.5 102.6) (layer B.SilkS)
+    (effects (font (size 0.65 0.6) (thickness 0.1)) (justify mirror))
+  )
+  (gr_text Power (at 116.5 102.4) (layer B.SilkS)
     (effects (font (size 1 1) (thickness 0.2)) (justify mirror))
   )
