File: hardware/STM32L0xx/STM32L0xx_18650.sch (KiCad schematic (older format))
At the start: 50 parts, among them J1 SW Debug, J2 Battery, J3 GPIO, J4 USB_B_Micro, J5 Power, J6 LEDs, J7 GPIO, Q1 BSS806N, Q2 BSS806N, Q3 BSS806N, Q4 BSS806N, SW1 Mode, SW2 Power, U1 STM32L072KZTx, U2 AP2210N-3.3TRG1, U3 MCP73833-AMI_UN, Y1 32.768kHz

Commit message: Convert 4 layer -> 2 layer PCB (#2)
Parts:
- removed J1: SW Debug, Connector_PinHeader_1.27mm:PinHeader_2x05_P1.27mm_Vertical, symbol Connector:Conn_ARM_JTAG_SWD_10
- C9: footprint Capacitor_SMD:C_0603_1608Metric_Pad1.05x0.95mm_HandSolder -> Capacitor_SMD:C_0603_1608Metric
- D4, D5, D7, D8: value LED_Small -> LED
- J7: footprint Connector_PinHeader_2.54mm:PinHeader_1x05_P2.54mm_Vertical -> Connector_PinHeader_2.54mm:PinHeader_1x08_P2.54mm_Vertical; symbol Connector_Generic:Conn_01x05 -> Connector_Generic:Conn_01x08
Connections:
- net PB5: now also J7.5 (Pin_5); no longer J7.3 (Pin_3)
- net PB6: now also J7.6 (Pin_6); no longer J7.4 (Pin_4)
- net PB7: now also J7.7 (Pin_7); no longer J7.5 (Pin_5)
- net RESET: now also J7.8 (Pin_8)
- net SWCLK renamed PA14
- net PA14: now also J7.4 (Pin_4)
- net SWDIO renamed PA13
- net PA13: now also J7.3 (Pin_3)
Other:
- note removed: "JTAG / SWD"
- moved on the sheet: J3, J5, U2
