File: hardware/Standard_18650/STM32L0xx_18650.sch (KiCad schematic (older format))
At the start: 53 parts, among them J2 Battery, J3 GPIO, J4 USB_B_Micro, J5 Power, J6 LEDs, J7 GPIO, Q1 BSS806N, Q2 BSS806N, Q3 BSS806N, Q4 BSS806N, SW1 Mode, SW2 Power, U1 STM32L072KZTx, U2 AP2210N-3.3TRG1, U3 BQ21040, U4 ESD7002WTT1G, Y1 32.768kHz

Commit message: Minor adjustments/text/icon
Parts:
- R11: value 430 -> 330
Changed lines of the file:
@@
 AR Path="/5DBBDA3F" Ref="R11"  Part="1"
 F 0 "R11" V 9680 5850 50  0000 C CNN
-F 1 "430" V 9600 5850 50  0000 C CNN
+F 1 "330" V 9600 5850 50  0000 C CNN
 F 2 "Resistor_SMD:R_0603_1608Metric" V 9530 5850 50  0001 C CNN
 F 3 "" H 9600 5850 50  0001 C CNN

Commit message: Use STM32F412CGUx (Regular & Tiny)
Parts:
- removed U1: STM32L072KZTx, Package_QFP:LQFP-32_7x7mm_P0.8mm, symbol MCU_ST_STM32L0:STM32L072KZTx
- added C14: 4.7uF, Capacitor_SMD:C_0603_1608Metric, symbol Device:C_Small
- added C15, C16: 100nf, Capacitor_SMD:C_0603_1608Metric, symbol Device:C_Small
- added U1: STM32F412CGUx, Package_DFN_QFN:QFN-48-1EP_7x7mm_P0.5mm_EP5.6x5.6mm, symbol MCU_ST_STM32F4:STM32F412CGUx
- C3: value 10nf -> 100nf
Connections:
- net labels added: VDDA, XTAL1, XTAL2
- wire segments 204 -> 220
- no-connect marks 5 -> 15
Other:
- note added: "VDDA Decoupling"
- moved on the sheet: C10, C2, C3, C4, C5, C7, C8, L1, Y1
