File: hardware/Standard_18650/18650.sch (KiCad schematic (older format))
At the start: 57 parts, among them J2 Battery, J3 GPIO, J4 USB_B_Micro, J5 Power, J6 LEDs, J7 GPIO, Q1 BSS806N, Q2 BSS806N, Q3 BSS806N, Q4 BSS806N, SW1 Mode, SW2 Power, U1 STM32F411CE, U2 AP2210N-3.3TRG1, U3 MCP73830, U4 ESD7002WTT1G, U5 GD25Q16CEIGR, Y1 24Mhz

Commit message: Checkpoint commit (v1.2a3)
Parts:
- SW2: footprint Jeremy:Switch_L068-A-DC30V1A -> Jeremy Button/Switch:SW_KAN-15_PHT; MPN L068-A -> LG-15F
Changed lines of the file:
@@
 F 0 "SW2" H 1300 1575 50  0000 C CNN
 F 1 "Power" H 1300 1350 50  0000 C CNN
-F 2 "Jeremy:Switch_L068-A-DC30V1A" H 1300 1450 50  0001 C CNN
-F 3 "https://www.aliexpress.com/item/32966597068.html" H 1300 1450 50  0001 C CNN
-F 4 "L068-A" H 1300 1450 60  0001 C CNN "MPN"
+F 2 "Jeremy Button/Switch:SW_KAN-15_PHT" H 1300 1450 50  0001 C CNN
+F 3 "https://www.aliexpress.com/item/32965072924.html" H 1300 1450 50  0001 C CNN
+F 4 "LG-15F" H 1300 1450 60  0001 C CNN "MPN"
 	1    1300 1450
 	1    0    0    -1

Commit message: Circuit updates
Parts:
- J4: symbol Connector:USB_B_Micro -> 18650-rescue:USB_B_Micro-Connector
Changed lines of the file:
@@
 $EndDescr
 $Comp
-L Connector:USB_B_Micro J4
+L 18650-rescue:USB_B_Micro-Connector J4
 U 1 1 5BD51321
 P 2800 6850
