File: hardware/Tiny_10440/10440.kicad_pcb (KiCad board)
At the start: 2 copper layers, 87.5 x 16 mm, 51 parts, among them J2 Battery, J3 GPIO, J4 USB_B_Micro, J5 LEDs, J7 GPIO/Power, Q1 BSS806N, Q2 BSS806N, Q3 BSS806N, Q4 BSS806N, SW1 Mode, SW2 Power, U1 STM32F412CGUx, U2 AP2210N-3.3TRG1, U3 MCP73831T-2ACI_OT, U4 ESD7002WTT1G

Commit message: Update gerbers
Parts:
- moved D4 2.81 mm to (99.2, 93.6)
- moved D5 2.70 mm to (96.1, 93.6)
- moved J5 2.65 mm to (101.8, 96.2)
- moved D7 2.62 mm to (93.0, 93.6)
- moved D8 2.58 mm to (89.8, 93.6)
- moved J3 0.81 mm to (84.4, 93.6)
- moved J7 0.81 mm to (74.3, 106.3)
- moved Q1 0.76 mm to (101.5, 101.2)
- moved Q2 0.75 mm to (98.7, 101.2)
- moved Q3 0.75 mm to (95.7, 101.2)
- moved Q4 0.75 mm to (92.7, 101.2)
- moved R10 0.75 mm to (95.1, 98.7)
- moved R12 0.75 mm to (91.9, 98.7)
- moved R7 0.75 mm to (101.5, 98.7)
- moved R8 0.75 mm to (98.3, 98.7)
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Routing:
- net GND: track 23.1 -> 30.8 mm, vias 2 -> 0
- net +BATT: track 25.1 -> 21.0 mm
- net Net-(D5-Pad1): track 2.61 -> 6.23 mm
- net Net-(D7-Pad1): track 2.71 -> 6.21 mm
- net Net-(D4-Pad1): track 2.50 -> 5.99 mm
- net Net-(D8-Pad1): track 2.77 -> 6.19 mm
- net +3V3: track 32.6 -> 35.6 mm, vias 10 -> 9
- net /LED1: track 7.64 -> 4.92 mm
- net /LED4: track 6.55 -> 4.44 mm
- net /LED3: track 6.94 -> 4.83 mm
- net /LED2: track 6.90 -> 4.82 mm
- net /PWM2: track 14.7 -> 16.4 mm
- net /PA13: track 7.98 -> 6.38 mm
- net /PWM3: track 11.4 -> 12.9 mm
- net /PA10: track 8.50 -> 9.52 mm
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Other:
- board text added: "rev 1.2a"
- board text removed: "rev 1a"
