File: hardware/Small_14500/14500.sch (KiCad schematic (older format))
At the start: 54 parts, among them J2 Battery, J3 GPIO, J4 USB_B_Micro, J6 LEDs, J7 GPIO, Q1 BSS806N, Q2 BSS806N, Q3 BSS806N, Q4 BSS806N, SW1 Mode, SW2 Power, U1 STM32F412CGUx, U2 AP2210N-3.3TRG1, U3 MCP73831T-2ACI_OT, U4 ESD7002WTT1G, Y1 24Mhz

Commit message: Production boards.
Parts:
- C10, C14, C3, C4, C5: value 100nf -> 100nF
- C2: value 1uf -> 1uF
- R2: value 20K -> 20k
- R6: value 675 -> 680
- U1: value STM32F412CGUx -> STM32F411CEU6
Changed lines of the file:
@@
 P 5700 1700
 F 0 "C3" H 5800 1700 50  0000 L CNN
-F 1 "100nf" H 5700 1600 50  0000 L CNN
+F 1 "100nF" H 5700 1600 50  0000 L CNN
 F 2 "Capacitor_SMD:C_0603_1608Metric" H 5700 1700 50  0001 C CNN
 F 3 "~" H 5700 1700 50  0001 C CNN
@@
 P 5450 1700
 F 0 "C2" H 5250 1700 50  0000 L CNN
-F 1 "1uf" H 5450 1600 50  0000 L CNN
+F 1 "1uF" H 5450 1600 50  0000 L CNN
 F 2 "Capacitor_SMD:C_0603_1608Metric" H 5450 1700 50  0001 C CNN
 F 3 "~" H 5450 1700 50  0001 C CNN
@@
 AR Path="/5E4A0482" Ref="R2"  Part="1"
 F 0 "R2" V 1430 7200 50  0000 C CNN
-F 1 "20K" V 1350 7200 50  0000 C CNN
+F 1 "20k" V 1350 7200 50  0000 C CNN
 F 2 "Resistor_SMD:R_0603_1608Metric" V 1280 7200 50  0001 C CNN
 F 3 "" H 1350 7200 50  0001 C CNN
@@
 AR Path="/5E4A04AD" Ref="R6"  Part="1"
 F 0 "R6" H 8350 5550 50  0000 L CNN
-F 1 "675" H 8300 5450 50  0000 L CNN
+F 1 "680" H 8300 5450 50  0000 L CNN
 F 2 "Resistor_SMD:R_0603_1608Metric" H 8500 5500 50  0001 C CNN
 F 3 "" H 8500 5500 50  0001 C CNN
@@
 P 3750 3250
 F 0 "U1" H 4150 1650 50  0000 C CNN
-F 1 "STM32F412CGUx" H 3150 4850 50  0000 C CNN
+F 1 "STM32F411CEU6" H 3150 4850 50  0000 C CNN
 F 2 "Package_DFN_QFN:QFN-48-1EP_7x7mm_P0.5mm_EP5.6x5.6mm" H 3150 1750 50  0001 R CNN
 F 3 "http://www.st.com/st-web-ui/static/active/en/resource/technical/document/datasheet/DM00213872.pdf" H 3750 3250 50  0001 C CNN
@@
 P 4750 1300
 F 0 "C5" H 4750 1500 50  0000 L CNN
-F 1 "100nf" H 4750 1200 50  0000 L CNN
+F 1 "100nF" H 4750 1200 50  0000 L CNN
 F 2 "Capacitor_SMD:C_0603_1608Metric" H 4750 1300 50  0001 C CNN
 F 3 "~" H 4750 1300 50  0001 C CNN
@@
 P 4450 1300
 F 0 "C4" H 4450 1500 50  0000 L CNN
-F 1 "100nf" H 4450 1200 50  0000 L CNN
+F 1 "100nF" H 4450 1200 50  0000 L CNN
 F 2 "Capacitor_SMD:C_0603_1608Metric" H 4450 1300 50  0001 C CNN
 F 3 "~" H 4450 1300 50  0001 C CNN
@@
 P 4200 1300
 F 0 "C14" H 4150 1500 50  0000 L CNN
-F 1 "100nf" H 4200 1200 50  0000 L CNN
+F 1 "100nF" H 4200 1200 50  0000 L CNN
 F 2 "Capacitor_SMD:C_0603_1608Metric" H 4200 1300 50  0001 C CNN
 F 3 "~" H 4200 1300 50  0001 C CNN
@@
 P 3950 1300
 F 0 "C10" H 3900 1500 50  0000 L CNN
-F 1 "100nf" H 3950 1200 50  0000 L CNN
+F 1 "100nF" H 3950 1200 50  0000 L CNN
 F 2 "Capacitor_SMD:C_0603_1608Metric" H 3950 1300 50  0001 C CNN
 F 3 "~" H 3950 1300 50  0001 C CNN
