File: hardware/Compact/Compact.sch (KiCad schematic (older format))
At the start: 46 parts, among them J2 Battery, J3 GPIO, J4 USB_B_Micro, J6 LEDs, J7 GPIO, Q1 BSS806N, Q2 BSS806N, Q3 BSS806N, Q4 BSS806N, SW1 Mode, SW2 Power, U1 STM32F411CE, U2 AP2210N-3.3TRG1, U3 MCP73831T-2ACI_OT, U5 GD25Q16CEIGR, Y1 24Mhz

Commit message: Update switch footprint.
Parts:
- D1, D2: footprint Diode_SMD:D_SOD-323_HandSoldering -> Diode_SMD:D_SOD-323
- R1: value 270 -> 330
- R6: value 680 -> 2k
Connections:
- wire segments 207 -> 208
Changed lines of the file:
@@
 Text Notes 8200 4200 0    50   ~ 0
 Battery Charger
-Text Label 4300 6850 0    50   ~ 0
-USB_D+
-Text Label 4300 6950 0    50   ~ 0
-USB_D-
 $Comp
 L power:GND #PWR0107
@@
 F 0 "D1" V 900 1100 50  0000 R CNN
 F 1 "20V2A" V 850 1450 50  0000 R CNN
-F 2 "Diode_SMD:D_SOD-323_HandSoldering" V 850 1150 50  0001 C CNN
+F 2 "Diode_SMD:D_SOD-323" V 850 1150 50  0001 C CNN
 F 3 "~" V 850 1150 50  0001 C CNN
 F 4 "SMD22WS-TP" H 850 1150 50  0001 C CNN "MPN"
@@
 	0    -1   -1   0
 $EndComp
-Text Label 4300 6650 0    50   ~ 0
-VUSB
 $Comp
 L Jeremy:AP2210-3.3TRG1 U2
@@
 	2750 7350 2750 7400
 Wire Notes Line
-	4650 6350 4650 7700
-Wire Notes Line
-	2500 6350 4650 6350
-Wire Notes Line
-	2500 7700 4650 7700
-Wire Notes Line
 	2500 6350 2500 7700
 Wire Wire Line
 	3450 7050 3450 6650
-Connection ~ 3450 6650
-Wire Wire Line
-	3450 6650 4300 6650
 $Comp
 L power:GND #PWR0104
@@
 F 0 "D2" V 1100 1100 50  0000 R CNN
 F 1 "20V2A" V 1000 1100 50  0000 R CNN
-F 2 "Diode_SMD:D_SOD-323_HandSoldering" V 1050 1150 50  0001 C CNN
+F 2 "Diode_SMD:D_SOD-323" V 1050 1150 50  0001 C CNN
 F 3 "~" V 1050 1150 50  0001 C CNN
 F 4 "SMD22WS-TP" H 1050 1150 50  0001 C CNN "MPN"
@@
 AR Path="/5BF9E96B" Ref="R1"  Part="1"
 F 0 "R1" V 980 5950 50  0000 C CNN
-F 1 "270" V 900 5950 50  0000 C CNN
+F 1 "330" V 900 5950 50  0000 C CNN
 F 2 "Resistor_SMD:R_0603_1608Metric" V 830 5950 50  0001 C CNN
 F 3 "" H 900 5950 50  0001 C CNN
@@
 AR Path="/5F01DEFD" Ref="R6"  Part="1"
 F 0 "R6" H 9100 5100 50  0000 L CNN
-F 1 "680" H 9050 5000 50  0000 L CNN
+F 1 "2k" H 9100 5000 50  0000 L CNN
 F 2 "Resistor_SMD:R_0603_1608Metric" H 9250 5050 50  0001 C CNN
 F 3 "" H 9250 5050 50  0001 C CNN
@@
 	3650 1350 3850 1350
 Wire Wire Line
-	3100 6850 4300 6850
-Wire Wire Line
-	3100 6950 4300 6950
-Wire Wire Line
 	5900 4750 5900 4600
 Wire Wire Line
@@
 Wire Wire Line
 	3100 6650 3450 6650
+Connection ~ 3450 6650
+Wire Wire Line
+	2900 6650 3100 6650
+Text Label 3750 6650 0    50   ~ 0
+VUSB
+Text Label 3750 6950 0    50   ~ 0
+USB_D-
+Text Label 3750 6850 0    50   ~ 0
+USB_D+
+Connection ~ 3100 6650
+Wire Wire Line
+	3100 6850 3750 6850
+Wire Wire Line
+	3100 6950 3750 6950
+Wire Wire Line
+	3450 6650 3750 6650
+Wire Notes Line
+	2500 6350 4100 6350
+Wire Notes Line
+	4100 6350 4100 7700
+Wire Notes Line
+	4100 7700 2500 7700
 $EndSCHEMATC

Commit message: Add 4 PWM LEDs.
Parts:
- added D4, D5, D7, D8: LED, LED_SMD:LED_0603_1608Metric, symbol Device:LED_Small
- added JP1: Jumper, Jumper:SolderJumper-2_P1.3mm_Bridged_RoundedPad1.0x1.5mm, symbol Device:Jumper
- added R10, R12, R7, R8: 270, Resistor_SMD:R_0603_1608Metric, symbol Device:R_Small
- J4: symbol Connector:USB_B_Micro -> Compact-rescue:USB_B_Micro-Connector
- SW2: footprint Jeremy:Switch_LG-15F -> Jeremy Button/Switch:SW_KAN-15_SMD; MPN L068-A -> KAN15
Connections:
- wire segments 208 -> 231
Other:
- moved on the sheet: D3, R1
Changed lines of the file:
@@
 $EndDescr
 $Comp
-L Connector:USB_B_Micro J4
+L Compact-rescue:USB_B_Micro-Connector J4
 U 1 1 5BD51321
 P 2800 6850
@@
 L Device:R R?
 U 1 1 5BF9E96B
-P 900 5950
+P 1600 5950
 AR Path="/5BD64BD8/5BF9E96B" Ref="R?"  Part="1"
 AR Path="/5BF9E96B" Ref="R1"  Part="1"
-F 0 "R1" V 980 5950 50  0000 C CNN
-F 1 "330" V 900 5950 50  0000 C CNN
-F 2 "Resistor_SMD:R_0603_1608Metric" V 830 5950 50  0001 C CNN
-F 3 "" H 900 5950 50  0001 C CNN
-F 4 "0603" V 900 5950 50  0001 C CNN "Package"
-	1    900  5950
+F 0 "R1" V 1680 5950 50  0000 C CNN
+F 1 "330" V 1600 5950 50  0000 C CNN
+F 2 "Resistor_SMD:R_0603_1608Metric" V 1530 5950 50  0001 C CNN
+F 3 "" H 1600 5950 50  0001 C CNN
+F 4 "0603" V 1600 5950 50  0001 C CNN "Package"
+	1    1600 5950
 	0    1    1    0
 $EndComp
@@
 	700  5700 700  5950
 Wire Wire Line
-	1100 5950 1050 5950
-Wire Wire Line
-	1550 5950 1550 6050
-Wire Wire Line
-	1400 5950 1550 5950
+	1800 5950 1750 5950
+Wire Wire Line
+	2250 5950 2250 6050
+Wire Wire Line
+	2100 5950 2250 5950
 $Comp
 L power:GND #PWR?
 U 1 1 5BF9E963
-P 1550 6050
+P 2250 6050
 AR Path="/5BD64BD8/5BF9E963" Ref="#PWR?"  Part="1"
 AR Path="/5BF9E963" Ref="#PWR0128"  Part="1"
-F 0 "#PWR0128" H 1550 5800 50  0001 C CNN
-F 1 "GND" H 1550 5900 50  0000 C CNN
-F 2 "" H 1550 6050 50  0001 C CNN
-F 3 "" H 1550 6050 50  0001 C CNN
-	1    1550 6050
+F 0 "#PWR0128" H 2250 5800 50  0001 C CNN
+F 1 "GND" H 2250 5900 50  0000 C CNN
+F 2 "" H 2250 6050 50  0001 C CNN
+F 3 "" H 2250 6050 50  0001 C CNN
+	1    2250 6050
 	1    0    0    -1
 $EndComp
@@
 L Device:LED D?
 U 1 1 5BF9E95C
-P 1250 5950
+P 1950 5950
 AR Path="/5BD64BD8/5BF9E95C" Ref="D?"  Part="1"
 AR Path="/5BF9E95C" Ref="D3"  Part="1"
-F 0 "D3" H 1250 6050 50  0000 C CNN
-F 1 "LED" H 1250 5850 50  0000 C CNN
-F 2 "LED_SMD:LED_0603_1608Metric_Castellated" H 1250 5950 50  0001 C CNN
-F 3 "" H 1250 5950 50  0001 C CNN
-F 4 "150060SS75000" H 1250 5950 50  0001 C CNN "MPN"
-F 5 "0603" H -100 1700 50  0001 C CNN "Package"
-	1    1250 5950
+F 0 "D3" H 1950 6050 50  0000 C CNN
+F 1 "LED" H 1950 5850 50  0000 C CNN
+F 2 "LED_SMD:LED_0603_1608Metric_Castellated" H 1950 5950 50  0001 C CNN
+F 3 "" H 1950 5950 50  0001 C CNN
+F 4 "150060SS75000" H 1950 5950 50  0001 C CNN "MPN"
+F 5 "0603" H 600 1700 50  0001 C CNN "Package"
+	1    1950 5950
 	-1   0    0    1
 $EndComp
@@
 F 0 "SW2" H 1300 1575 50  0000 C CNN
 F 1 "Power" H 1300 1350 50  0000 C CNN
-F 2 "Jeremy:Switch_LG-15F" H 1300 1450 50  0001 C CNN
-F 3 "https://www.aliexpress.com/item/32966597068.html" H 1300 1450 50  0001 C CNN
-F 4 "L068-A" H 1300 1450 60  0001 C CNN "MPN"
+F 2 "Jeremy Button/Switch:SW_KAN-15_SMD" H 1300 1450 50  0001 C CNN
+F 3 "" H 1300 1450 50  0001 C CNN
+F 4 "KAN15" H 1300 1450 60  0001 C CNN "MPN"
 	1    1300 1450
 	1    0    0    -1
@@
 Wire Notes Line
 	4100 7700 2500 7700
+$Comp
+L Device:Jumper JP1
+U 1 1 5F90FCAF
+P 1050 5950
+F 0 "JP1" H 1050 5950 50  0000 C CNN
+F 1 "Jumper" H 1050 5850 50  0000 C CNN
+F 2 "Jumper:SolderJumper-2_P1.3mm_Bridged_RoundedPad1.0x1.5mm" H 1050 5950 50  0001 C CNN
+F 3 "~" H 1050 5950 50  0001 C CNN
+	1    1050 5950
+	1    0    0    -1
+$EndComp
+Wire Wire Line
+	1350 5950 1450 5950
+$Comp
+L Device:LED_Small D5
+U 1 1 5F9A5BBF
+P 8600 1050
+F 0 "D5" H 8600 1150 50  0000 C CNN
+F 1 "LED" H 8600 1194 50  0001 C CNN
+F 2 "LED_SMD:LED_0603_1608Metric" V 8600 1050 50  0001 C CNN
+F 3 "~" V 8600 1050 50  0001 C CNN
+F 4 "150060VS75000" H 8600 1050 50  0001 C CNN "MPN"
+F 5 "0603" H 50  -350 50  0001 C CNN "Package"
+	1    8600 1050
+	1    0    0    -1
+$EndComp
+$Comp
+L Device:R_Small R8
+U 1 1 5F9A5BC7
+P 8350 1050
+F 0 "R8" V 8250 1050 50  0000 C CNN
+F 1 "270" V 8350 1050 39  0000 C CNN
+F 2 "Resistor_SMD:R_0603_1608Metric" H 8350 1050 50  0001 C CNN
+F 3 "~" H 8350 1050 50  0001 C CNN
+F 4 "CRCW0603270RJNEA" H 8350 1050 50  0001 C CNN "MPN"
+F 5 "0603" H 50  -350 50  0001 C CNN "Package"
+	1    8350 1050
+	0    1    1    0
+$EndComp
+Wire Wire Line
+	8200 1050 8250 1050
+Wire Wire Line
+	8450 1050 8500 1050
+$Comp
+L Device:LED_Small D4
+U 1 1 5F9A5BD1
+P 7700 1050
+F 0 "D4" H 7700 1150 50  0000 C CNN
+F 1 "LED" H 7700 1194 50  0001 C CNN
+F 2 "LED_SMD:LED_0603_1608Metric" V 7700 1050 50  0001 C CNN
+F 3 "~" V 7700 1050 50  0001 C CNN
+F 4 "150060VS75000" H 7700 1050 50  0001 C CNN "MPN"
+F 5 "0603" H 50  -350 50  0001 C CNN "Package"
+	1    7700 1050
+	1    0    0    -1
+$EndComp
+Wire Wire Line
+	7300 1050 7350 1050
+Wire Wire Line
+	7550 1050 7600 1050
+$Comp
+L Device:LED_Small D7
+U 1 1 5F9A5BE3
+P 9500 1050
+F 0 "D7" H 9500 1150 50  0000 C CNN
+F 1 "LED" H 9500 1194 50  0001 C CNN
+F 2 "LED_SMD:LED_0603_1608Metric" V 9500 1050 50  0001 C CNN
+F 3 "~" V 9500 1050 50  0001 C CNN
+F 4 "150060VS75000" H 9500 1050 50  0001 C CNN "MPN"
+F 5 "0603" H 50  -350 50  0001 C CNN "Package"
+	1    9500 1050
+	1    0    0    -1
+$EndComp
+$Comp
+L Device:R_Small R10
+U 1 1 5F9A5BEB
+P 9250 1050
+F 0 "R10" V 9150 1050 50  0000 C CNN
+F 1 "270" V 9250 1050 39  0000 C CNN
+F 2 "Resistor_SMD:R_0603_1608Metric" H 9250 1050 50  0001 C CNN
+F 3 "~" H 9250 1050 50  0001 C CNN
+F 4 "CRCW0603270RJNEA" H 9250 1050 50  0001 C CNN "MPN"
+F 5 "0603" H 50  -350 50  0001 C CNN "Package"
+	1    9250 1050
+	0    1    1    0
+$EndComp
+Wire Wire Line
+	9350 1050 9400 1050
+$Comp
+L Device:LED_Small D8
+U 1 1 5F9A5BF4
+P 10300 1050
+F 0 "D8" H 10300 1150 50  0000 C CNN
+F 1 "LED" H 10300 1194 50  0001 C CNN
+F 2 "LED_SMD:LED_0603_1608Metric" V 10300 1050 50  0001 C CNN
+F 3 "~" V 10300 1050 50  0001 C CNN
+F 4 "150060VS75000" H 10300 1050 50  0001 C CNN "MPN"
+F 5 "0603" H 50  -350 50  0001 C CNN "Package"
+	1    10300 1050
+	1    0    0    -1
+$EndComp
+$Comp
+L Device:R_Small R12
+U 1 1 5F9A5BFC
+P 10050 1050
+F 0 "R12" V 9950 1050 50  0000 C CNN
+F 1 "270" V 10050 1050 39  0000 C CNN
+F 2 "Resistor_SMD:R_0603_1608Metric" H 10050 1050 50  0001 C CNN
+F 3 "~" H 10050 1050 50  0001 C CNN
+F 4 "CRCW0603270RJNEA" H 10050 1050 50  0001 C CNN "MPN"
+F 5 "0603" H 50  -350 50  0001 C CNN "Package"
+	1    10050 1050
+	0    1    1    0
+$EndComp
+Wire Wire Line
+	9900 1050 9950 1050
+Wire Wire Line
+	10150 1050 10200 1050
+Wire Wire Line
+	9050 1050 9150 1050
+$Comp
+L power:+3.3V #PWR03
+U 1 1 5F9A5C05
+P 8950 800
+F 0 "#PWR03" H 8950 650 50  0001 C CNN
+F 1 "+3.3V" H 8965 973 50  0000 C CNN
+F 2 "" H 8950 800 50  0001 C CNN
+F 3 "" H 8950 800 50  0001 C CNN
+	1    8950 800
+	1    0    0    -1
+$EndComp
+Wire Wire Line
+	7800 1050 7950 1050
+Wire Wire Line
+	7300 1250 7300 1050
+Wire Wire Line
+	8200 1050 8200 1350
+Wire Wire Line
+	9050 1050 9050 1450
+Wire Wire Line
+	9900 1050 9900 1550
+Wire Wire Line
+	7950 1050 7950 800
+Wire Wire Line
+	7950 800  8850 800
+Wire Wire Line
+	8700 1050 8850 1050
+Wire Wire Line
+	8850 1050 8850 800
+Connection ~ 8850 800
+Wire Wire Line
+	8850 800  8950 800
+Wire Wire Line
+	9600 1050 9600 800
+Wire Wire Line
+	9600 800  8950 800
+Connection ~ 8950 800
+Wire Wire Line
+	10400 1050 10400 800
+Wire Wire Line
+	10400 800  9600 800
+Connection ~ 9600 800
+Connection ~ 7300 1250
+Connection ~ 8200 1350
+Connection ~ 9050 1450
+Connection ~ 9900 1550
+$Comp
+L Device:R_Small R7
+U 1 1 5F9A5BD9
+P 7450 1050
+F 0 "R7" V 7350 1050 50  0000 C CNN
+F 1 "270" V 7450 1050 39  0000 C CNN
+F 2 "Resistor_SMD:R_0603_1608Metric" H 7450 1050 50  0001 C CNN
+F 3 "~" H 7450 1050 50  0001 C CNN
+F 4 "CRCW0603270RJNEA" H 7450 1050 50  0001 C CNN "MPN"
+F 5 "0603" H 50  -350 50  0001 C CNN "Package"
+	1    7450 1050
+	0    1    1    0
+$EndComp
 $EndSCHEMATC

Commit message: Circuit updates
Parts:
- D9: footprint LED_SMD:LED-APA102-2020 -> Jeremy LEDs:LED-APA102-2020
- R10, R12, R7, R8: value 270 -> 330
- R6: MPN (none) -> RMCF0603FT2K00
Changed lines of the file:
@@
 F 0 "D9" H 10250 3100 50  0000 C CNN
 F 1 "APA102-2020" H 10800 3100 50  0000 C CNN
-F 2 "LED_SMD:LED-APA102-2020" H 10500 3100 50  0001 L TNN
+F 2 "Jeremy LEDs:LED-APA102-2020" H 10500 3100 50  0001 L TNN
 F 3 "https://cdn.sparkfun.com/assets/0/1/5/c/3/_20181120__APA_102-2020-256-8.pdf" H 10550 3025 50  0001 L TNN
 	1    10450 3400
@@
 F 3 "" H 9250 5050 50  0001 C CNN
 F 4 "0603" H 900 -450 50  0001 C CNN "Package"
+F 5 "RMCF0603FT2K00" H 9250 5050 50  0001 C CNN "MPN"
 	1    9250 5050
 	1    0    0    -1
@@
 P 8350 1050
 F 0 "R8" V 8250 1050 50  0000 C CNN
-F 1 "270" V 8350 1050 39  0000 C CNN
+F 1 "330" V 8350 1050 39  0000 C CNN
 F 2 "Resistor_SMD:R_0603_1608Metric" H 8350 1050 50  0001 C CNN
 F 3 "~" H 8350 1050 50  0001 C CNN
@@
 P 9250 1050
 F 0 "R10" V 9150 1050 50  0000 C CNN
-F 1 "270" V 9250 1050 39  0000 C CNN
+F 1 "330" V 9250 1050 39  0000 C CNN
 F 2 "Resistor_SMD:R_0603_1608Metric" H 9250 1050 50  0001 C CNN
 F 3 "~" H 9250 1050 50  0001 C CNN
@@
 P 10050 1050
 F 0 "R12" V 9950 1050 50  0000 C CNN
-F 1 "270" V 10050 1050 39  0000 C CNN
+F 1 "330" V 10050 1050 39  0000 C CNN
 F 2 "Resistor_SMD:R_0603_1608Metric" H 10050 1050 50  0001 C CNN
 F 3 "~" H 10050 1050 50  0001 C CNN
@@
 P 7450 1050
 F 0 "R7" V 7350 1050 50  0000 C CNN
-F 1 "270" V 7450 1050 39  0000 C CNN
+F 1 "330" V 7450 1050 39  0000 C CNN
 F 2 "Resistor_SMD:R_0603_1608Metric" H 7450 1050 50  0001 C CNN
 F 3 "~" H 7450 1050 50  0001 C CNN

Commit message: Minor updates
Parts:
- U2: symbol Jeremy:AP2210-3.3TRG1 -> Compact-rescue:AP2210-3.3TRG1-Jeremy
- U3: symbol dk_PMIC-Battery-Chargers:MCP73831T-2ACI_OT -> DigiKey-Battery:MCP73831T-2ACI_OT
- U5: symbol Jeremy:GD25Q16CEIGR -> Compact-rescue:GD25Q16CEIGR-Jeremy
Changed lines of the file:
@@
 $EndComp
 $Comp
-L Jeremy:AP2210-3.3TRG1 U2
+L Compact-rescue:AP2210-3.3TRG1-Jeremy U2
 U 1 1 5CD3E552
 P 5650 6950
@@
 Connection ~ 8850 3400
 $Comp
-L Jeremy:GD25Q16CEIGR U5
+L Compact-rescue:GD25Q16CEIGR-Jeremy U5
 U 1 1 5F002A37
 P 8100 3450
@@
 	10450 4800 10600 4800
 $Comp
-L dk_PMIC-Battery-Chargers:MCP73831T-2ACI_OT U3
+L DigiKey-Battery:MCP73831T-2ACI_OT U3
 U 1 1 5F2441F8
 P 9650 4800
