File: hardware/Original/Original.sch (KiCad schematic (older format))
At the start: 57 parts, among them J2 Battery, J3 GPIO, J4 USB_B_Micro, J5 Power, J6 LEDs, J7 GPIO, Q1 BSS806N, Q2 BSS806N, Q3 BSS806N, Q4 BSS806N, SW1 Mode, SW2 Power, U1 STM32F411CE, U2 AP2210N-3.3TRG1, U3 MCP73830, U4 ESD7002WTT1G, U5 GD25Q16CEIGR, Y1 24Mhz

Commit message: Update KAN15 LED placement.
Parts:
- J4: symbol 18650-rescue:USB_B_Micro-Connector -> Connector:USB_B_Micro
Changed lines of the file:
@@
 $EndDescr
 $Comp
-L 18650-rescue:USB_B_Micro-Connector J4
+L Connector:USB_B_Micro J4
 U 1 1 5BD51321
 P 2800 6850

Commit message: Add ESD. Update labeling
Parts:
- U2: symbol Jeremy:AP2210-3.3TRG1 -> Original-rescue:AP2210-3.3TRG1-Jeremy
- U3: symbol jg_Battery_Management:MCP73830 -> Original-rescue:MCP73830-jg_Battery_Management
- U4: symbol Jeremy:ESD7002WTT1G -> Original-rescue:ESD7002WTT1G-Jeremy
- U5: symbol Jeremy:GD25Q16CEIGR -> Original-rescue:GD25Q16CEIGR-Jeremy
Changed lines of the file:
@@
 VUSB
 $Comp
-L Jeremy:AP2210-3.3TRG1 U2
+L Original-rescue:AP2210-3.3TRG1-Jeremy U2
 U 1 1 5CD3E552
 P 5650 6950
@@
 	3100 6950 3800 6950
 $Comp
-L Jeremy:ESD7002WTT1G U4
+L Original-rescue:ESD7002WTT1G-Jeremy U4
 U 1 1 5DA9EA0D
 P 4200 7300
@@
 	1    0    0    -1
 $EndComp
-Connection ~ 3850 1350
-Wire Wire Line
-	3550 1350 3850 1350
 Wire Wire Line
 	3650 1850 3650 1750
-Wire Wire Line
-	3850 1350 4100 1350
 Connection ~ 4100 1350
 Wire Wire Line
-	3850 1550 3850 1600
-Wire Wire Line
-	3850 1600 4100 1600
-Wire Wire Line
 	4100 1550 4100 1600
-Connection ~ 4100 1600
 Connection ~ 4400 1350
 Wire Wire Line
@@
 Wire Wire Line
 	2150 2700 1750 2700
-$Comp
-L Device:C_Small C15
-U 1 1 5E4C30F8
-P 3850 1450
-F 0 "C15" H 3900 1450 50  0000 L CNN
-F 1 "100nF" H 3850 1350 50  0000 L CNN
-F 2 "Capacitor_SMD:C_0603_1608Metric" H 3850 1450 50  0001 C CNN
-F 3 "~" H 3850 1450 50  0001 C CNN
-F 4 "AVX" H 3850 1450 50  0001 C CNN "MFN"
-F 5 "06035C104K4T2A" H 3850 1450 50  0001 C CNN "MPN"
-F 6 "0603" H -500 -250 50  0001 C CNN "Package"
-	1    3850 1450
-	1    0    0    -1
-$EndComp
 NoConn ~ 3100 7050
 $Comp
@@
 Connection ~ 8850 4050
 $Comp
-L Jeremy:GD25Q16CEIGR U5
+L Original-rescue:GD25Q16CEIGR-Jeremy U5
 U 1 1 5F002A37
 P 8100 4100
@@
 	3750 6850 4300 6850
 $Comp
-L jg_Battery_Management:MCP73830 U3
+L Original-rescue:MCP73830-jg_Battery_Management U3
 U 1 1 5F52DFD0
 P 9700 5600
@@
 	1    0    0    -1
 $EndComp
+Wire Wire Line
+	3850 1550 3850 1600
+Connection ~ 4100 1600
+Wire Wire Line
+	3850 1600 4100 1600
+Wire Wire Line
+	3850 1350 4100 1350
+Wire Wire Line
+	3550 1350 3850 1350
+Connection ~ 3850 1350
+$Comp
+L Device:C_Small C15
+U 1 1 5E4C30F8
+P 3850 1450
+F 0 "C15" H 3900 1450 50  0000 L CNN
+F 1 "100nF" H 3850 1350 50  0000 L CNN
+F 2 "Capacitor_SMD:C_0603_1608Metric" H 3850 1450 50  0001 C CNN
+F 3 "~" H 3850 1450 50  0001 C CNN
+F 4 "AVX" H 3850 1450 50  0001 C CNN "MFN"
+F 5 "06035C104K4T2A" H 3850 1450 50  0001 C CNN "MPN"
+F 6 "0603" H -500 -250 50  0001 C CNN "Package"
+	1    3850 1450
+	1    0    0    -1
+$EndComp
